Commit message: Update antenna z-height in URDF

File: olav_description/urdf/descriptions/olav.urdf (robot description, URDF)
Before this commit: robot olav, 17 links, 16 joints
Joints:
- joint gnss_ins_to_gnss_ins_antenna_1_fixed: origin xyz=+0.6038 +0.4229 +0.2503 rpy=+0.0 +0.0 +0.0 -> xyz=+0.6038 +0.4229 +0.451 rpy=+0.0 +0.0 +0.0
- joint gnss_ins_to_gnss_ins_antenna_2_fixed: origin xyz=+0.6038 -0.7043 +0.2503 rpy=+0.0 +0.0 +0.0 -> xyz=+0.6038 -0.7043 +0.451 rpy=+0.0 +0.0 +0.0

Commit message: Fix URDF antenna position

File: olav_description/urdf/descriptions/olav.urdf (robot description, URDF)
Before this commit: robot olav, 17 links, 16 joints
Joints:
- joint gnss_ins_to_gnss_ins_antenna_1_fixed: origin xyz=+0.6038 +0.4229 +0.2503 rpy=+0.0 +0.0 +0.0 -> xyz=+0.6038 -0.7043 +0.451 rpy=+0.0 +0.0 +0.0

Commit message: Fix URDF antenna positions

File: olav_description/urdf/descriptions/olav.urdf (robot description, URDF)
Before this commit: robot olav, 17 links, 16 joints
Joints:
- joint gnss_ins_to_gnss_ins_antenna_1_fixed: origin xyz=+0.6038 -0.7043 +0.451 rpy=+0.0 +0.0 +0.0 -> xyz=+0.6038 +0.4229 +0.451 rpy=+0.0 +0.0 +0.0

Commit message: Update URDF transforms

File: olav_description/urdf/descriptions/olav.urdf (robot description, URDF)
Before this commit: robot olav, 17 links, 16 joints
Joints:
- joint base_to_camera_top_fixed: origin xyz=+1.1898 -0.1231 +0.5781 rpy=+0.0000 +0.00872665 +0.0000 -> xyz=+1.1898 -0.1231 +0.5781 rpy=+3.14159 +0.0087 +0.0000
- joint gnss_ins_to_gnss_ins_antenna_1_fixed: origin xyz=+0.6038 +0.4229 +0.451 rpy=+0.0 +0.0 +0.0 -> xyz=+0.6038 +0.3876 +0.451 rpy=+0.0 +0.0 +0.0
- joint gnss_ins_to_gnss_ins_antenna_2_fixed: origin xyz=+0.6038 -0.7043 +0.451 rpy=+0.0 +0.0 +0.0 -> xyz=+0.6038 -0.6924 +0.451 rpy=+0.0 +0.0 +0.0
